File: Kicad_Ultrasonic_Speaker/ultrasonic array/ultrasonic array.kicad_sch (KiCad schematic)
At the start: 37 parts, among them J1 Screw_Terminal_01x02_from_cir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

Commit message: change kicad
Parts:
- J1: value Screw_Terminal_01x02_from_circuit -> Screw_Terminal_01x02
