File: Kicad_Ultrasonic_Speaker/ultrasonic array/ultrasonic array.kicad_pcb (KiCad board)
At the start: 2 copper layers, 111.3 x 93 mm, 37 parts, among them J1 Screw_Terminal_01x02_from_cir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

Commit message: change kicad
Parts:
- J1: value Screw_Terminal_01x02_from_circuit -> Screw_Terminal_01x02

Commit message: try flatCAM
Other:
- board size 111.3 x 93 mm -> 116.8 x 96.5 mm
Changed lines of the file:
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@@
     )
     (pad_to_mask_clearance 0)
+    (aux_axis_origin 137.929047 131.509642)
     (pcbplotparams
-      (layerselection 0x0001000_ffffffff)
+      (layerselection 0x0001080_7fffffff)
       (plot_on_all_layers_selection 0x0000000_00000000)
       (disableapertmacros false)
@@
       (viasonmask false)
       (mode 1)
-      (useauxorigin false)
+      (useauxorigin true)
       (hpglpennumber 1)
       (hpglpenspeed 20)
@@
     )
   )
-  (gr_poly
-    (pts
-      (arc (start 103.234486 132.741342) (mid 104.698952 136.276876) (end 108.234486 137.741342))
-      (arc (start 209.534486 137.741342) (mid 213.07002 136.276876) (end 214.534486 132.741342))
-      (arc (start 214.534486 49.741342) (mid 213.07002 46.205808) (end 209.534486 44.741342))
-      (arc (start 108.234486 44.741342) (mid 104.698952 46.205808) (end 103.234486 49.741342))
-    )
-    (stroke (width 0.2) (type solid)) (fill none) (layer "Edge.Cuts"))
+  (gr_rect (start 101.6 43.18) (end 218.44 139.7)
+    (stroke (width 0.1) (type default)) (fill none) (layer "Edge.Cuts"))
   (segment (start 114.9 95.857359) (end 114.9 94.45) (width 1) (layer "F.Cu") (net 1))
   (segment (start 109.209209 71.701534) (end 113.997172 71.701534) (width 1) (layer "F.Cu") (net 1))
